File: Hardware/KiCad/Cryologger GVMS/Cryologger GVMS.sch (KiCad schematic (older format))
At the start: 12 parts, among them J1 Screw_Terminal_01x02, J2 Screw_Terminal_01x02, U1 MMDLCB, U2 POLOLU_DV36, U3 GPS-RTK-SMA

Commit message: Update KiCad files
Parts:
- removed J2: Screw_Terminal_01x02, TerminalBlock_Phoenix:TerminalBlock_Phoenix_PT-1,5-2-5.0-H_1x02_P5.00mm_Horizontal, symbol Connector:Screw_Terminal_01x02
- J1: footprint TerminalBlock_Phoenix:TerminalBlock_Phoenix_PT-1,5-2-5.0-H_1x02_P5.00mm_Horizontal -> Connector_Phoenix_MSTB:PhoenixContact_MSTBA_2,5_2-G-5,08_1x02_P5.08mm_Horizontal
- U1: footprint Cryologger GVMS:MMDLCB -> Cryologger:SparkFun_MMDLCB
- U2: footprint Cryologger GVMS:POLOLU_DV36 -> Cryologger:Pololu_D36V6
- U3: footprint Cryologger GVMS:GPS-RTK-SMA -> Cryologger:SparkFun_GPS-RTK-SMA
Connections:
- net labels added: +5V
- net labels removed: LOAD, VBAT, VOUT
- wire segments 67 -> 58
Other:
- moved on the sheet: J1, U2
Changed lines of the file:
@@
 Text Notes 4150 900  0    79   ~ 16
 Power Management
-$Comp
-L power:GND #PWR04
-U 1 1 60777168
-P 4550 1800
-F 0 "#PWR04" H 4550 1550 50  0001 C CNN
-F 1 "GND" H 4555 1627 50  0000 C CNN
-F 2 "" H 4550 1800 50  0001 C CNN
-F 3 "" H 4550 1800 50  0001 C CNN
-	1    4550 1800
-	1    0    0    -1
-$EndComp
-$Comp
-L power:GND #PWR03
-U 1 1 60777821
-P 5450 1750
-F 0 "#PWR03" H 5450 1500 50  0001 C CNN
-F 1 "GND" H 5455 1577 50  0000 C CNN
-F 2 "" H 5450 1750 50  0001 C CNN
-F 3 "" H 5450 1750 50  0001 C CNN
-	1    5450 1750
-	1    0    0    -1
-$EndComp
-Wire Wire Line
-	4500 1700 4550 1700
-Wire Wire Line
-	4550 1700 4550 1800
 Text Label 1250 5000 2    50   ~ 0
 SDA
@@
 Wire Wire Line
 	2600 5500 2800 5500
-Text Label 5600 1600 2    50   ~ 0
-VBAT
-Text Label 4750 1600 2    50   ~ 0
-LOAD
 Wire Notes Line
 	600  600  3550 600
@@
 Wire Wire Line
 	2650 2550 2650 3250
-Wire Wire Line
-	2600 2250 2650 2250
-Wire Wire Line
-	2650 2250 2650 2150
-Wire Wire Line
-	2650 1950 2600 1950
-Wire Wire Line
-	2600 2050 2650 2050
-Connection ~ 2650 2050
-Wire Wire Line
-	2650 2050 2650 1950
-Wire Wire Line
-	2600 2150 2650 2150
-Connection ~ 2650 2150
-Wire Wire Line
-	2650 2150 2650 2050
-Wire Wire Line
-	2650 1950 2750 1950
-Connection ~ 2650 1950
 $Comp
 L power:GND #PWR05
@@
 $EndComp
 Wire Wire Line
-	5400 1700 5450 1700
-Wire Wire Line
-	5450 1700 5450 1750
-Wire Wire Line
-	2000 3350 2050 3350
-Connection ~ 2050 3350
-Wire Wire Line
-	2050 3350 2100 3350
-Text Label 2050 3550 1    50   ~ 0
-VOUT
-Wire Wire Line
-	2050 3350 2050 3550
+	2000 3350 2000 3550
 Wire Wire Line
 	6900 1700 6600 1700
@@
 L power:GND #PWR06
 U 1 1 60889145
-P 5100 3150
-F 0 "#PWR06" H 5100 2900 50  0001 C CNN
-F 1 "GND" H 5105 2977 50  0000 C CNN
-F 2 "" H 5100 3150 50  0001 C CNN
-F 3 "" H 5100 3150 50  0001 C CNN
-	1    5100 3150
+P 5000 3050
+F 0 "#PWR06" H 5000 2800 50  0001 C CNN
+F 1 "GND" H 5005 2877 50  0000 C CNN
+F 2 "" H 5000 3050 50  0001 C CNN
+F 3 "" H 5000 3050 50  0001 C CNN
+	1    5000 3050
 	1    0    0    -1
 $EndComp
@@
 F 0 "U3" H 1975 4627 50  0000 C CNN
 F 1 "GPS-RTK-SMA" H 1975 4536 50  0000 C CNN
-F 2 "Cryologger GVMS:GPS-RTK-SMA" H 1750 5250 50  0001 C CNN
+F 2 "Cryologger:SparkFun_GPS-RTK-SMA" H 1750 5250 50  0001 C CNN
 F 3 "" H 1750 5250 50  0001 C CNN
 	1    2000 5250
@@
 F 0 "U1" H 2050 3515 50  0000 C CNN
 F 1 "MMDLCB" H 2050 3424 50  0000 C CNN
-F 2 "Cryologger GVMS:MMDLCB" H 1950 2800 50  0001 C CNN
+F 2 "Cryologger:SparkFun_MMDLCB" H 1950 2800 50  0001 C CNN
 F 3 "" H 1950 2800 50  0001 C CNN
 	1    2050 2350
@@
 L Cryologger_GVMS:POLOLU_DV36 U2
 U 1 1 60758F09
-P 4700 2850
-F 0 "U2" H 4758 3265 50  0000 C CNN
-F 1 "POLOLU_DV36" H 4758 3174 50  0000 C CNN
-F 2 "Cryologger GVMS:POLOLU_DV36" H 4600 2800 50  0001 C CNN
-F 3 "" H 4600 2800 50  0001 C CNN
-	1    4700 2850
-	1    0    0    -1
-$EndComp
-Wire Wire Line
-	5050 2800 5100 2800
-Wire Wire Line
-	5100 2800 5100 3150
-Wire Wire Line
-	5050 2700 5100 2700
-Wire Wire Line
-	5100 2700 5100 2550
-Wire Wire Line
-	5050 2900 5200 2900
-Wire Wire Line
-	5200 2900 5200 2550
-Text Label 5100 2550 1    50   ~ 0
-VOUT
-Text Label 5200 2550 1    50   ~ 0
-LOAD
+P 4600 2750
+F 0 "U2" H 4658 3165 50  0000 C CNN
+F 1 "POLOLU_DV36" H 4658 3074 50  0000 C CNN
+F 2 "Cryologger:Pololu_D36V6" H 4500 2700 50  0001 C CNN
+F 3 "" H 4500 2700 50  0001 C CNN
+	1    4600 2750
+	1    0    0    -1
+$EndComp
+Wire Wire Line
+	4950 2700 5000 2700
+Wire Wire Line
+	5000 2700 5000 3050
+Wire Wire Line
+	4950 2600 5000 2600
+Wire Wire Line
+	5000 2600 5000 2450
+Wire Wire Line
+	4950 2800 5200 2800
+Wire Wire Line
+	5200 2800 5200 2450
 $Comp
 L Mechanical:MountingHole_Pad H1
@@
 	1    0    0    -1
 $EndComp
-$Comp
-L Connector:Screw_Terminal_01x02 J2
-U 1 1 6075F22F
-P 5200 1700
-F 0 "J2" H 5118 1375 50  0000 C CNN
-F 1 "Screw_Terminal_01x02" H 5118 1466 50  0000 C CNN
-F 2 "TerminalBlock_Phoenix:TerminalBlock_Phoenix_PT-1,5-2-5.0-H_1x02_P5.00mm_Horizontal" H 5200 1700 50  0001 C CNN
-F 3 "~" H 5200 1700 50  0001 C CNN
-	1    5200 1700
-	-1   0    0    1
-$EndComp
 Wire Notes Line
 	7700 600  7700 2700
@@
 Mounting Holes
 $Comp
-L power:+3V3 #PWR?
+L power:+3V3 #PWR0101
 U 1 1 607AB278
 P 2750 4650
-F 0 "#PWR?" H 2750 4500 50  0001 C CNN
+F 0 "#PWR0101" H 2750 4500 50  0001 C CNN
 F 1 "+3V3" H 2765 4823 50  0000 C CNN
 F 2 "" H 2750 4650 50  0001 C CNN
@@
 Wire Wire Line
 	2750 5000 2750 4650
-$Comp
-L power:+3V3 #PWR?
-U 1 1 607B0868
-P 2750 1350
-F 0 "#PWR?" H 2750 1200 50  0001 C CNN
-F 1 "+3V3" H 2765 1523 50  0000 C CNN
-F 2 "" H 2750 1350 50  0001 C CNN
-F 3 "" H 2750 1350 50  0001 C CNN
-	1    2750 1350
-	1    0    0    -1
-$EndComp
-Wire Wire Line
-	2750 1950 2750 1350
 Text Notes 1050 4200 0    79   ~ 16
 SparkFun GPS-RTK-SMA ZED-F9P\n
 Connection ~ 6750 2200
 $Comp
-L power:+BATT #PWR?
+L power:+BATT #PWR0102
 U 1 1 60939999
 P 6900 1200
-F 0 "#PWR?" H 6900 1050 50  0001 C CNN
+F 0 "#PWR0102" H 6900 1050 50  0001 C CNN
 F 1 "+BATT" H 6915 1373 50  0000 C CNN
 F 2 "" H 6900 1200 50  0001 C CNN
@@
 	1    0    0    -1
 $EndComp
+Wire Wire Line
+	8000 1300 8000 1500
+Connection ~ 8000 1500
+Wire Wire Line
+	8000 1500 8000 1700
+Connection ~ 8000 1700
+Wire Wire Line
+	8000 1700 8000 1900
+Connection ~ 8000 1900
+Wire Wire Line
+	8000 1900 8000 2050
+Wire Wire Line
+	1500 2400 1400 2400
+Wire Wire Line
+	1400 2400 1400 1350
+$Comp
+L power:+3V3 #PWR0103
+U 1 1 608A03EA
+P 1400 1350
+F 0 "#PWR0103" H 1400 1200 50  0001 C CNN
+F 1 "+3V3" H 1415 1523 50  0000 C CNN
+F 2 "" H 1400 1350 50  0001 C CNN
+F 3 "" H 1400 1350 50  0001 C CNN
+	1    1400 1350
+	1    0    0    -1
+$EndComp
+$Comp
+L power:GND #PWR04
+U 1 1 60777168
+P 4800 1800
+F 0 "#PWR04" H 4800 1550 50  0001 C CNN
+F 1 "GND" H 4805 1627 50  0000 C CNN
+F 2 "" H 4800 1800 50  0001 C CNN
+F 3 "" H 4800 1800 50  0001 C CNN
+	1    4800 1800
+	1    0    0    -1
+$EndComp
+Wire Wire Line
+	4800 1700 4800 1800
+Wire Wire Line
+	4750 1700 4800 1700
+Wire Wire Line
+	4750 1600 4800 1600
 $Comp
 L Connector:Screw_Terminal_01x02 J1
 U 1 1 60760DDE
-P 4300 1700
-F 0 "J1" H 4218 1375 50  0000 C CNN
-F 1 "Screw_Terminal_01x02" H 4218 1466 50  0000 C CNN
-F 2 "TerminalBlock_Phoenix:TerminalBlock_Phoenix_PT-1,5-2-5.0-H_1x02_P5.00mm_Horizontal" H 4300 1700 50  0001 C CNN
-F 3 "~" H 4300 1700 50  0001 C CNN
-	1    4300 1700
+P 4550 1700
+F 0 "J1" H 4468 1375 50  0000 C CNN
+F 1 "Screw_Terminal_01x02" H 4468 1466 50  0000 C CNN
+F 2 "Connector_Phoenix_MSTB:PhoenixContact_MSTBA_2,5_2-G-5,08_1x02_P5.08mm_Horizontal" H 4550 1700 50  0001 C CNN
+F 3 "~" H 4550 1700 50  0001 C CNN
+	1    4550 1700
 	-1   0    0    1
 $EndComp
 Wire Wire Line
-	5400 1600 5600 1600
-Wire Wire Line
-	4500 1600 4750 1600
-Wire Wire Line
-	8000 1300 8000 1500
-Connection ~ 8000 1500
-Wire Wire Line
-	8000 1500 8000 1700
-Connection ~ 8000 1700
-Wire Wire Line
-	8000 1700 8000 1900
-Connection ~ 8000 1900
-Wire Wire Line
-	8000 1900 8000 2050
+	4800 1400 4800 1600
+$Comp
+L power:+BATT #PWR0104
+U 1 1 609AB5FC
+P 4800 1400
+F 0 "#PWR0104" H 4800 1250 50  0001 C CNN
+F 1 "+BATT" H 4815 1573 50  0000 C CNN
+F 2 "" H 4800 1400 50  0001 C CNN
+F 3 "" H 4800 1400 50  0001 C CNN
+	1    4800 1400
+	1    0    0    -1
+$EndComp
+$Comp
+L power:+BATT #PWR0105
+U 1 1 609B6114
+P 5200 2450
+F 0 "#PWR0105" H 5200 2300 50  0001 C CNN
+F 1 "+BATT" H 5215 2623 50  0000 C CNN
+F 2 "" H 5200 2450 50  0001 C CNN
+F 3 "" H 5200 2450 50  0001 C CNN
+	1    5200 2450
+	1    0    0    -1
+$EndComp
+$Comp
+L power:+5V #PWR0106
+U 1 1 609B737B
+P 5000 2450
+F 0 "#PWR0106" H 5000 2300 50  0001 C CNN
+F 1 "+5V" H 5015 2623 50  0000 C CNN
+F 2 "" H 5000 2450 50  0001 C CNN
+F 3 "" H 5000 2450 50  0001 C CNN
+	1    5000 2450
+	1    0    0    -1
+$EndComp
+$Comp
+L power:+5V #PWR0107
+U 1 1 609BE5A5
+P 2200 3550
+F 0 "#PWR0107" H 2200 3400 50  0001 C CNN
+F 1 "+5V" H 2215 3723 50  0000 C CNN
+F 2 "" H 2200 3550 50  0001 C CNN
+F 3 "" H 2200 3550 50  0001 C CNN
+	1    2200 3550
+	1    0    0    -1
+$EndComp
+Connection ~ 2000 3350
+Wire Wire Line
+	2000 3350 2100 3350
+Wire Wire Line
+	2000 3550 2200 3550
 $EndSCHEMATC
